File: electronic_scale.kicad_sch (KiCad schematic)
At the start: 0 parts

Commit message: 更正电源开关电路的原理错误
Other:
- note added: "拉低关机"
- note removed: "拉高关机"
Changed lines of the file:
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@@
 		)
 	)
-	(text "拉高关机"
+	(text "拉低关机"
 		(exclude_from_sim no)
 		(at 123.952 95.758 0)
